File: kicad/ckt-autointchg/ckt-autointchg.kicad_sch (KiCad schematic)
At the start: 22 parts, among them J1 Screw_Terminal_01x02, J2 Screw_Terminal_01x02, J3 Screw_Terminal_01x02, J4 Conn_AVR_TagConnect_TC2030, Q1 BSS138, SW1 FSM4JSMATR, SW2 SW_DIP_x05, U1 MC78L05_SOT89, U2 ATtiny13A-S, U2A1 ATtiny13A-SS

Commit message: Finished schematic
Parts:
- added H1, H2, H3, H4: MountingHole, MountingHole:MountingHole_3.2mm_M3_Pad, symbol Mechanical:MountingHole_Pad
- added J5: Conn_01x02_Male, Connector_PinHeader_2.54mm:PinHeader_1x02_P2.54mm_Vertical, symbol Connector:Conn_01x02_Male
- added RLY1: 3570-1419-05x, ISE_UltraLibrarian:3570.1419.054, symbol ISE_UltraLibrarian:Comus_3570
- added RLY2: 3570-1331-05x, ISE_UltraLibrarian:3570-1331-051, symbol ISE_UltraLibrarian:Comus_3570
Connections:
- net GND: now also J5.2 (Pin_2)
- net at D3.1 (K), D4.2 (A), Q1.3 (D): now also RLY1.3, RLY2.3
- net at D1.4, J1.2 (Pin_2): now also RLY1.1, RLY2.1
- net at C2.1, C3.1, D4.1 (K)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: now also RLY1.2, RLY2.2
- net at J4.5 (~{RESET}), R1.1, SW1.1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: now also J5.1 (Pin_1)
- net at J2.1 (Pin_1): now also RLY1.4, RLY2.4
Other:
- note added: "DCC A"
- note added: "DCC B"
- note added: "IR GND (black)"
- note added: "IR IN (white)"
- note added: "IR PWR (red)"
- note added: "N.C."
- note added: "Switched DCC B"
- moved on the sheet: C1, C2, C3, C4, D1, D2, D3, D4, J1, J2, J3, J4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
